Commit message: Update change base_link to pivot

File: whill_description/whill_model_cr2.urdf (robot description, URDF)
Before this commit: robot whill_model_cr2, 12 links, 11 joints
Links:
- link base_link: geometry visual cylinder length=0.2 radius=0.01
Joints:
- joint base_floor_joint: origin xyz=0 0 0 rpy=0 0 0 -> xyz=0.3 0 0 rpy=0 0 0
