Commit message: 最初のコミット

File: whill_description/urdf/body/whill_model_cr2.urdf.xacro (robot description, xacro)
@@ -1,4 +1,8 @@
 <?xml version="1.0"?>
-<robot name="whill_model_cr2">
+<robot name="${robot_name}" xmlns:xacro="http://ros.org/wiki/xacro">
+  <xacro:arg name="robot_name" default="whill_model_cr2"/>
+  <!-- もし Gazebo 切り替えを使うなら下も -->
+  <xacro:arg name="gazebo" default="classic"/>
+  <xacro:arg name="use_ros2_control" default="false"/>
     <link name="base_link">
         <visual>
@@ -283,4 +287,10 @@
         <origin xyz="0 -0.245 0.30" rpy="0 1.0 0"/>
     </joint>
+    <xacro:include filename="$(find whill_description)/urdf/lider/lider.urdf.xacro"/>
+    <xacro:lrf_v0 prefix="front" parent="backrest">
+      <joint_origin>
+        <origin xyz="0.1 0.25 " rpy="0 0 0"/>
+      </joint_origin>
+    </xacro:lrf_v0>
     <!-- Diff Drive Plugin -->
     <gazebo>

File: whill_description/urdf/lider/lider.urdf.xacro (robot description, xacro)
@@ -1,7 +1,7 @@
 <?xml version="1.0"?>
 <robot xmlns:xacro="http://ros.org/wiki/xacro">
-  <xacro:include filename="$(find ros2_whill)/whill_description/urdf/common.xacro"/>
-  <xacro:include filename="$(find ros2_whill)/whill_description/urdf/lider/lider.gazebo.xacro"/>
-  <xacro:macro name="lrf_v0" params="prefix parent *joint_origin">
+  <xacro:include filename="$(find whill_description)/urdf/common.xacro"/>
+  <xacro:include filename="$(find whill_description)/urdf/lider/lider.gazebo.xacro"/>
+  <xacro:macro name="lrf_v0" params="prefix parent *backrest">
     <joint name="${prefix}_lrf_joint" type="fixed">
       <xacro:insert_block name="joint_origin"/>
@@ -12,10 +12,10 @@
       <visual>
         <geometry>
-          <mesh filename="file://$(find ros2_whill)/whill_description/model/meshes/dae/lrf.dae"/>
+          <mesh filename="file://$(find whill_description)/model/meshes/dae/lrf.dae"/>
         </geometry>
       </visual>
       <collision>
         <geometry>
-          <mesh filename="file://$(find ros2_whill)/whill_description/model/meshes/stl/lrf.stl"/>
+          <mesh filename="file://$(find whill_description)/model/meshes/stl/lrf.stl"/>
         </geometry>
       </collision>

Commit message: ディレクトリ整理(launch未作成)

File: whill_description/urdf/body/whill_model_cr2.urdf.xacro (robot description, xacro)
@@ -1,314 +1,285 @@
 <?xml version="1.0"?>
-<robot name="${robot_name}" xmlns:xacro="http://ros.org/wiki/xacro">
-  <xacro:arg name="robot_name" default="whill_model_cr2"/>
-  <!-- もし Gazebo 切り替えを使うなら下も -->
-  <xacro:arg name="gazebo" default="classic"/>
-  <xacro:arg name="use_ros2_control" default="false"/>
-    <link name="base_link">
-        <visual>
-            <geometry>
-                <cylinder length="0.2" radius="0.01"/>
-            </geometry>
-            <material name="blue">
-                <color rgba="0.0 0.0 1.0 1.0"/>
-            </material>
-        </visual>
-    </link>
-    <link name="base_floor">
-        <visual>
-            <geometry>
-                <box size="0.985 0.37 0.03"/>
-            </geometry>
-            <material name="grey">
-                <color rgba="0.5 0.5 0.5 1.0"/>
-            </material>
-        </visual>
-        <collision>
-            <geometry>
-                <box size="0.985 0.37 0.03"/>
-            </geometry>
-        </collision>
-        <inertial>
-            <origin xyz="0 0 0" rpy="0 0 0" />
-            <mass value="30" />
-            <inertia ixx="1.0"  ixy="0.0"   ixz="0.0"
-                                iyy="1.0"   iyz="0.0"
-                                            izz="1.0" />
-        </inertial>
-    </link>
-    <joint name="base_floor_joint" type="fixed">
-        <parent link="base_link" />
-        <child link="base_floor" />
-        <origin xyz="0.3 0 0" rpy="0 0 0"/>
-    </joint>
-    <link name="left_wheel">
-        <visual>
-            <geometry>
-                <cylinder length="0.05" radius="0.1325"/>
-            </geometry>
-            <origin xyz="0 0 0" rpy="0 0 0" />
-            <material name="black">
-                <color rgba="0.1 0.1 0.1 1.0"/>
-            </material>
-        </visual>
-        <collision>
-            <geometry>
-                <cylinder length="0.05" radius="0.1325"/>
-            </geometry>
-        </collision>
-        <inertial>
-            <origin xyz="0 0 0"/>
-            <mass value="0.500"/>
-            <inertia ixx="0.0013541667" ixy="0" ixz="0" iyy="0.0013541667" iyz="0" izz="0.0025"/>
-        </inertial>
-    </link>
-    <joint name="left_wheel_joint" type="continuous">
-        <parent link="base_floor" />
-        <child link="left_wheel" />
-        <origin xyz="-0.3 0.260 0.015" rpy="1.571 0 0" />
-        <axis xyz="0 0 1" />
-    </joint>
-    <link name="right_wheel">
-        <collision>
-            <origin xyz="0 0 0" rpy="0 0 0" />
-            <geometry>
-                <cylinder length="0.05" radius="0.1325"/>
-            </geometry>
-        </collision>
-        <visual>
-            <origin xyz="0 0 0" rpy="0 0 0" />
-            <geometry>
-                <cylinder length="0.05" radius="0.1325"/>
-            </geometry>
-            <material name="black">
-                <color rgba="0.1 0.1 0.1 1.0"/>
-            </material>
-        </visual>
-        <inertial>
-            <origin xyz="0 0 0"/>
-            <mass value="0.500"/>
-            <inertia ixx="0.0013541667" ixy="0" ixz="0" iyy="0.0013541667" iyz="0" izz="0.0025"/>
-        </inertial>
-    </link>
-    <joint name="right_wheel_joint" type="continuous">
-        <parent link="base_floor" />
-        <child link="right_wheel" />
-        <origin xyz="-0.3 -0.260 0.015" rpy="-1.571 0 0" />
-        <axis xyz="0 0 -1" />
-    </joint>
-    <link name="left_front_wheel">
-        <collision>
-            <geometry>
-                <cylinder length="0.05" radius="0.1325"/>
-            </geometry>
-        </collision>
-        <visual>
-            <geometry>
-                <cylinder length="0.05" radius="0.1325"/>
-            </geometry>
-            <material name="black">
-                <color rgba="0.1 0.1 0.1 1.0"/>
-            </material>
-        </visual>
-        <inertial>
-            <origin xyz="0 0 0" rpy="0 0 0" />
-            <mass value="1.0" />
-            <inertia ixx="1.0"  ixy="0.0"   ixz="0.0"
-                                iyy="1.0"   iyz="0.0"
-                                            izz="1.0" />
-        </inertial>
-    </link>
-    <joint name="left_front_wheel_joint" type="continuous">
-        <parent link="base_floor" />
-        <child link="left_front_wheel" />
-        <origin xyz="0.330 -0.235 0" rpy="-1.571 0 0" />
-        <axis xyz="0 0 -1" />
-    </joint>
-    <link name="right_front_wheel">
-        <collision>
-            <geometry>
-                <cylinder length="0.05" radius="0.1325"/>
-            </geometry>
-        </collision>
-        <visual>
-            <geometry>
-                <cylinder length="0.05" radius="0.1325"/>
-            </geometry>
-            <material name="black">
-                <color rgba="0.1 0.1 0.1 1.0"/>
-            </material>
-        </visual>
-        <inertial>
-            <origin xyz="0 0 0" rpy="0 0 0" />
-            <mass value="1.0" />
-            <inertia ixx="1.0"  ixy="0.0"   ixz="0.0"
-                                iyy="1.0"   iyz="0.0"
-                                            izz="1.0" />
-        </inertial>
-    </link>
-    <joint name="right_front_wheel_joint" type="continuous">
-        <parent link="base_floor" />
-        <child link="right_front_wheel"/>
-        <origin xyz="0.330 0.235 0" rpy="1.571 0 0" />
-        <axis xyz="0 0 1" />
-    </joint>
-    <link name="seat">
-        <visual>
-            <geometry>
-                <box size="0.42 0.42 0.40"/>
-            </geometry>
-            <material name="grey">
-                <color rgba="0.5 0.5 0.5 1.0"/>
-            </material>
-        </visual>
-        <collision>
-            <geometry>
-                <box size="0.42 0.42 0.40"/>
-            </geometry>
-        </collision>
-        <inertial>
-            <origin xyz="0 0 0" rpy="0 0 0" />
-            <mass value="12" />
-            <inertia ixx="1.0"  ixy="0.0"   ixz="0.0"
-                                iyy="1.0"   iyz="0.0"
-                                            izz="1.0" />
-        </inertial>
-    </link>
-    <joint name="seat_joint" type="fixed">
-        <parent link="base_floor" />
-        <child link="seat" />
-        <origin xyz="-0.10 0 0.215" rpy="0 0 0"/>
-    </joint>
-    <link name="left_sensor_arm">
-        <collision>
-            <geometry>
-                <cylinder length="0.11" radius="0.013"/>
-            </geometry>
-        </collision>
-        <visual>
-            <geometry>
-                <cylinder length="0.11" radius="0.013"/>
-            </geometry>
-            <material name="grey">
-                <color rgba="0.5 0.5 0.5 1.0"/>
-            </material>
-        </visual>
-    </link>
-    <joint name="left_sensor_arm_joint" type="fixed">
-        <parent link="seat"/>
-        <child link="left_sensor_arm"/>
-        <origin xyz="0.20 0.235 0.07" rpy="0 0 0"/>
-    </joint>
-    <link name="right_sensor_arm">
-        <collision>
-            <geometry>
-                <cylinder length="0.11" radius="0.013"/>
-            </geometry>
-        </collision>
-        <visual>
-            <geometry>
-                <cylinder length="0.11" radius="0.013"/>
-            </geometry>
-            <material name="grey">
-                <color rgba="0.5 0.5 0.5 1.0"/>
-            </material>
-        </visual>
-    </link>
-    <joint name="right_sensor_arm_joint" type="fixed">
-        <parent link="seat"/>
-        <child link="right_sensor_arm"/>
-        <origin xyz="0.20 -0.235 0.07" rpy="0 0 0"/>
-    </joint>
-    <link name="backrest">
-        <visual>
-            <geometry>
-                <box size="0.10 0.42 0.72"/>
-            </geometry>
-            <material name="grey">
-                <color rgba="0.5 0.5 0.5 1.0"/>
-            </material>
-        </visual>
-        <collision>
-            <geometry>
-                <box size="0.10 0.42 0.72"/>
-            </geometry>
-        </collision>
-        <inertial>
-            <origin xyz="0 0 0" rpy="0 0 0" />
-            <mass value="7" />
-            <inertia ixx="1.0"  ixy="0.0"   ixz="0.0"
-                                iyy="1.0"   iyz="0.0"
-                                            izz="1.0" />
-        </inertial>
-    </link>
-    <joint name="backrest_joint" type="fixed">
-        <parent link="base_floor" />
-        <child link="backrest" />
-        <origin xyz="-0.36 0 0.375" rpy="0 0 0"/>
-    </joint>
-    <link name="left_arm">
-        <visual>
-            <geometry>
-                <box size="0.09 0.07 0.535"/>
-            </geometry>
-            <material name="grey">
-                <color rgba="0.5 0.5 0.5 1.0"/>
-            </material>
-        </visual>
-        <collision>
-            <geometry>
-                <box size="0.09 0.07 0.535"/>
-            </geometry>
-        </collision>
-    </link>
-    <joint name="left_arm_joint" type="fixed">
-        <parent link="seat" />
-        <child link="left_arm" />
-        <origin xyz="0 0.245 0.30" rpy="0 1.0 0"/>
-    </joint>
-    <link name="right_arm">
-        <visual>
-            <geometry>
-                <box size="0.09 0.07 0.535"/>
-            </geometry>
-            <material name="grey">
-                <color rgba="0.5 0.5 0.5 1.0"/>
-            </material>
-        </visual>
-        <collision>
-            <geometry>
-                <box size="0.09 0.07 0.535"/>
-            </geometry>
-        </collision>
-    </link>
-    <joint name="right_arm_joint" type="fixed">
-        <parent link="seat" />
-        <child link="right_arm" />
-        <origin xyz="0 -0.245 0.30" rpy="0 1.0 0"/>
-    </joint>
-    <xacro:include filename="$(find whill_description)/urdf/lider/lider.urdf.xacro"/>
-    <xacro:lrf_v0 prefix="front" parent="backrest">
-      <joint_origin>
-        <origin xyz="0.1 0.25 " rpy="0 0 0"/>
-      </joint_origin>
-    </xacro:lrf_v0>
-    <!-- Diff Drive Plugin -->
-    <gazebo>
-      <plugin
-        filename="libgz-sim-diff-drive-system.so"
-        name="gz::sim::systems::DiffDrive">
-        <!-- 左右車輪のジョイント名 -->
-        <left_joint>left_wheel_joint</left_joint>
-        <right_joint>right_wheel_joint</right_joint>
-        <!-- 制御するトピック名 -->
-        <topic>cmd_vel</topic>
-        <!-- エンコーダのフィードバック -->
-        <odom_topic>odom</odom_topic>
-        <odom_frame>odom</odom_frame>
-        <base_frame>base_link</base_frame>
-        <!-- ホイールのパラメータ（適宜修正してください） -->
-        <wheel_separation>0.45</wheel_separation>
-        <wheel_radius>0.1</wheel_radius>
-      </plugin>
-    </gazebo>
-</robot>
+<!-- whill_model_cr2: body-only definition (macroized). This file contains *only* links/joints.
+Place at: <your_package>/urdf/whill_model_cr2.urdf.xacro -->
+<xacro:macro name="whill_body_v0" params="robot_name='whill_model_cr2' gazebo='classic' use_ros2_control='false'">
+<xacro:arg name="robot_name" default="${robot_name}"/>
+<xacro:arg name="gazebo" default="${gazebo}"/>
+<xacro:arg name="use_ros2_control" default="${use_ros2_control}"/>
+<!-- Base link -->
+<link name="base_link">
+<visual>
+<geometry>
+<cylinder length="0.2" radius="0.01"/>
+</geometry>
+<material name="blue">
+<color rgba="0.0 0.0 1.0 1.0"/>
+</material>
+</visual>
+</link>
+<!-- Base floor -->
+<link name="base_floor">
+<visual>
+<geometry>
+<box size="0.985 0.37 0.03"/>
+</geometry>
+<material name="grey">
+<color rgba="0.5 0.5 0.5 1.0"/>
+</material>
+</visual>
+<collision>
+<geometry>
+<box size="0.985 0.37 0.03"/>
+</geometry>
+</collision>
+<inertial>
+<origin xyz="0 0 0" rpy="0 0 0" />
+<mass value="30" />
+<inertia ixx="1.0" ixy="0.0" ixz="0.0"
+iyy="1.0" iyz="0.0"
+izz="1.0" />
+</inertial>
+</link>
+<joint name="base_floor_joint" type="fixed">
+<parent link="base_link" />
+<child link="base_floor" />
+<origin xyz="0.3 0 0" rpy="0 0 0"/>
+</joint>
+<!-- Wheels (left/right + front) -->
+<link name="left_wheel">
+<visual>
+<geometry>
+<cylinder length="0.05" radius="0.1325"/>
+</geometry>
+<origin xyz="0 0 0" rpy="0 0 0" />
+<material name="black">
+<color rgba="0.1 0.1 0.1 1.0"/>
+</material>
+</visual>
+<collision>
+<geometry>
+<cylinder length="0.05" radius="0.1325"/>
+</geometry>
+</collision>
+<inertial>
+<origin xyz="0 0 0"/>
+<mass value="0.500"/>
+<inertia ixx="0.0013541667" ixy="0" ixz="0" iyy="0.0013541667" iyz="0" izz="0.0025"/>
+</inertial>
+</link>
+<joint name="left_wheel_joint" type="continuous">
+<parent link="base_floor" />
+<child link="left_wheel" />
+<origin xyz="-0.3 0.260 0.015" rpy="1.571 0 0" />
+<axis xyz="0 0 1" />
+</joint>
+<link name="right_wheel">
+<collision>
+<origin xyz="0 0 0" rpy="0 0 0" />
+<geometry>
+<cylinder length="0.05" radius="0.1325"/>
+</geometry>
+</collision>
+<visual>
+<origin xyz="0 0 0" rpy="0 0 0" />
+<geometry>
+<cylinder length="0.05" radius="0.1325"/>
+</geometry>
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
File: whill_description/urdf/lider/lider.urdf.xacro (robot description, xacro)
@@ -1,28 +1,43 @@
-<?xml version="1.0"?>
-<robot xmlns:xacro="http://ros.org/wiki/xacro">
-  <xacro:include filename="$(find whill_description)/urdf/common.xacro"/>
-  <xacro:include filename="$(find whill_description)/urdf/lider/lider.gazebo.xacro"/>
-  <xacro:macro name="lrf_v0" params="prefix parent *backrest">
-    <joint name="${prefix}_lrf_joint" type="fixed">
-      <xacro:insert_block name="joint_origin"/>
-      <parent link="${parent}"/>
-      <child link="${prefix}_lrf_link"/>
-    </joint>
-    <link name="${prefix}_lrf_link">
-      <visual>
-        <geometry>
-          <mesh filename="file://$(find whill_description)/model/meshes/dae/lrf.dae"/>
-        </geometry>
-      </visual>
-      <collision>
-        <geometry>
-          <mesh filename="file://$(find whill_description)/model/meshes/stl/lrf.stl"/>
-        </geometry>
-      </collision>
-      <inertial>
-        <origin xyz="0 0 0"/>
-        <xacro:box_inertial mass="0.218" height="0.07" width="0.05" depth="0.05"/>
-      </inertial>
-    </link>
-  </xacro:macro>
-</robot>
+--- file: urdf/lider/lider.urdf.xacro ---
+<!-- lider: standalone lidar macro. Place at: <your_package>/urdf/lider/lider.urdf.xacro -->
+<xacro:macro name="lrf_v0" params="prefix='front' parent='base_link' min_rad='-3.14' max_rad='3.14' min_range='0.06' max_range='10.0' gazebo='classic'">
+<!-- link for lidar -->
+<link name="${prefix}_lrf_link">
+<visual>
+<origin xyz="0 0 0" rpy="0 0 0"/>
+<geometry>
+<cylinder length="0.02" radius="0.03"/>
+</geometry>
+</visual>
+</link>
+<joint name="${prefix}_lrf_joint" type="fixed">
+<parent link="${parent}"/>
+<child link="${prefix}_lrf_link"/>
+<!-- joint_origin can be overridden by nested <joint_origin> in robot_top -->
+<origin xyz="0 0 0" rpy="0 0 0"/>
+</joint>
+<!-- Gazebo sensor (classic) -->
+<xacro:if value="${gazebo == 'classic'}">
+<gazebo reference="${prefix}_lrf_link">
+<sensor type="ray" name="${prefix}_laser">
+<update_rate>20</update_rate>
+<ray>
+<scan>
+<horizontal>
+<samples>360</samples>
+<resolution>1</resolution>
+</horizontal>
+</scan>
+<range>
+<min>${min_range}</min>
+<max>${max_range}</max>
+</range>
+</ray>
+<plugin name="${prefix}_gazebo_laser_plugin" filename="libgazebo_ros_range.so">
+<topicName>/${prefix}/scan</topicName>
+</plugin>
+</sensor>
+</gazebo>
+</xacro:if>
+<!-- Ignition/Garden sensor could be added here (omitted for brevity) -->
+</xacro:macro>
