Commit message: xacro→urdf展開エラーの修正+gazeboビルドエラーの修正

File: whill_description/urdf/body/whill_model_cr2.urdf.xacro (robot description, xacro)
@@ -1,285 +1,241 @@
 <?xml version="1.0"?>
-<!-- whill_model_cr2: body-only definition (macroized). This file contains *only* links/joints.
-Place at: <your_package>/urdf/whill_model_cr2.urdf.xacro -->
-<xacro:macro name="whill_body_v0" params="robot_name='whill_model_cr2' gazebo='classic' use_ros2_control='false'">
-<xacro:arg name="robot_name" default="${robot_name}"/>
-<xacro:arg name="gazebo" default="${gazebo}"/>
-<xacro:arg name="use_ros2_control" default="${use_ros2_control}"/>
-<!-- Base link -->
-<link name="base_link">
-<visual>
-<geometry>
-<cylinder length="0.2" radius="0.01"/>
-</geometry>
-<material name="blue">
-<color rgba="0.0 0.0 1.0 1.0"/>
-</material>
-</visual>
-</link>
-<!-- Base floor -->
-<link name="base_floor">
-<visual>
-<geometry>
-<box size="0.985 0.37 0.03"/>
-</geometry>
-<material name="grey">
-<color rgba="0.5 0.5 0.5 1.0"/>
-</material>
-</visual>
-<collision>
-<geometry>
-<box size="0.985 0.37 0.03"/>
-</geometry>
-</collision>
-<inertial>
-<origin xyz="0 0 0" rpy="0 0 0" />
-<mass value="30" />
-<inertia ixx="1.0" ixy="0.0" ixz="0.0"
-iyy="1.0" iyz="0.0"
-izz="1.0" />
-</inertial>
-</link>
-<joint name="base_floor_joint" type="fixed">
-<parent link="base_link" />
-<child link="base_floor" />
-<origin xyz="0.3 0 0" rpy="0 0 0"/>
-</joint>
-<!-- Wheels (left/right + front) -->
-<link name="left_wheel">
-<visual>
-<geometry>
-<cylinder length="0.05" radius="0.1325"/>
-</geometry>
-<origin xyz="0 0 0" rpy="0 0 0" />
-<material name="black">
-<color rgba="0.1 0.1 0.1 1.0"/>
-</material>
-</visual>
-<collision>
-<geometry>
-<cylinder length="0.05" radius="0.1325"/>
-</geometry>
-</collision>
-<inertial>
-<origin xyz="0 0 0"/>
-<mass value="0.500"/>
-<inertia ixx="0.0013541667" ixy="0" ixz="0" iyy="0.0013541667" iyz="0" izz="0.0025"/>
-</inertial>
-</link>
-<joint name="left_wheel_joint" type="continuous">
-<parent link="base_floor" />
-<child link="left_wheel" />
-<origin xyz="-0.3 0.260 0.015" rpy="1.571 0 0" />
-<axis xyz="0 0 1" />
-</joint>
-<link name="right_wheel">
-<collision>
-<origin xyz="0 0 0" rpy="0 0 0" />
-<geometry>
-<cylinder length="0.05" radius="0.1325"/>
-</geometry>
-</collision>
-<visual>
-<origin xyz="0 0 0" rpy="0 0 0" />
-<geometry>
-<cylinder length="0.05" radius="0.1325"/>
-</geometry>
-<material name="black">
-<color rgba="0.1 0.1 0.1 1.0"/>
-</material>
-</visual>
-<inertial>
-<origin xyz="0 0 0"/>
-<mass value="0.500"/>
-<inertia ixx="0.0013541667" ixy="0" ixz="0" iyy="0.0013541667" iyz="0" izz="0.0025"/>
-</inertial>
-</link>
-<joint name="right_wheel_joint" type="continuous">
-<parent link="base_floor" />
-<child link="right_wheel" />
-<origin xyz="-0.3 -0.260 0.015" rpy="-1.571 0 0" />
-<axis xyz="0 0 -1" />
-</joint>
-<!-- Front wheels -->
-<link name="left_front_wheel">
-<collision>
-<geometry>
-<cylinder length="0.05" radius="0.1325"/>
-</geometry>
-</collision>
-<visual>
-<geometry>
-<cylinder length="0.05" radius="0.1325"/>
-</geometry>
-<material name="black">
-<color rgba="0.1 0.1 0.1 1.0"/>
-</material>
-</visual>
-<inertial>
-<origin xyz="0 0 0" rpy="0 0 0" />
-<mass value="1.0" />
-<inertia ixx="1.0" ixy="0.0" ixz="0.0"
-iyy="1.0" iyz="0.0"
-izz="1.0" />
-</inertial>
-</link>
-<joint name="left_front_wheel_joint" type="continuous">
-<parent link="base_floor" />
-<child link="left_front_wheel" />
-<origin xyz="0.330 -0.235 0" rpy="-1.571 0 0" />
-<axis xyz="0 0 -1" />
-</joint>
-<link name="right_front_wheel">
-<collision>
-<geometry>
-<cylinder length="0.05" radius="0.1325"/>
-</geometry>
-</collision>
-<visual>
-<geometry>
-<cylinder length="0.05" radius="0.1325"/>
-</geometry>
-<material name="black">
-<color rgba="0.1 0.1 0.1 1.0"/>
-</material>
-</visual>
-<inertial>
-<origin xyz="0 0 0" rpy="0 0 0" />
-<mass value="1.0" />
-<inertia ixx="1.0" ixy="0.0" ixz="0.0"
-iyy="1.0" iyz="0.0"
-izz="1.0" />
-</inertial>
-</link>
-<joint name="right_front_wheel_joint" type="continuous">
-<parent link="base_floor" />
-<child link="right_front_wheel"/>
-<origin xyz="0.330 0.235 0" rpy="1.571 0 0" />
-<axis xyz="0 0 1" />
-</joint>
-<!-- Seat, arms, backrest -->
-<link name="seat">
-<visual>
-<geometry>
-<box size="0.42 0.42 0.40"/>
-</geometry>
-<material name="grey">
-<color rgba="0.5 0.5 0.5 1.0"/>
-</material>
-</visual>
-<collision>
-<geometry>
-<box size="0.42 0.42 0.40"/>
-</geometry>
-</collision>
-<inertial>
-<origin xyz="0 0 0" rpy="0 0 0" />
-<mass value="12" />
-<inertia ixx="1.0" ixy="0.0" ixz="0.0"
-iyy="1.0" iyz="0.0"
-izz="1.0" />
-</inertial>
-</link>
-<joint name="seat_joint" type="fixed">
-<parent link="base_floor" />
-<child link="seat" />
-<origin xyz="-0.10 0 0.215" rpy="0 0 0"/>
-</joint>
-<link name="left_sensor_arm">
-<collision>
-<geometry>
-<cylinder length="0.11" radius="0.013"/>
-</geometry>
-</collision>
-<visual>
-<geometry>
-<cylinder length="0.11" radius="0.013"/>
-</geometry>
-<material name="grey">
-<color rgba="0.5 0.5 0.5 1.0"/>
-</material>
-</visual>
-</link>
-<joint name="left_sensor_arm_joint" type="fixed">
-<geometry>
-<cylinder length="0.11" radius="0.013"/>
-</geometry>
-</collision>
-<visual>
-<geometry>
-<cylinder length="0.11" radius="0.013"/>
-</geometry>
-<material name="grey">
-<color rgba="0.5 0.5 0.5 1.0"/>
-</material>
-</visual>
-</link>
-<joint name="right_sensor_arm_joint" type="fixed">
-<parent link="seat"/>
-<child link="right_sensor_arm"/>
-<origin xyz="0.20 -0.235 0.07" rpy="0 0 0"/>
-</joint>
-<link name="backrest">
-<visual>
-<geometry>
-<box size="0.10 0.42 0.72"/>
-</geometry>
-<material name="grey">
-<color rgba="0.5 0.5 0.5 1.0"/>
-</material>
-</visual>
-<collision>
-<geometry>
-<box size="0.10 0.42 0.72"/>
-</geometry>
-</collision>
-<inertial>
-<origin xyz="0 0 0" rpy="0 0 0" />
-<mass value="7" />
-<inertia ixx="1.0" ixy="0.0" ixz="0.0"
-iyy="1.0" iyz="0.0"
-izz="1.0" />
-</inertial>
-</link>
-<joint name="backrest_joint" type="fixed">
-<visual>
-<geometry>
-<box size="0.09 0.07 0.535"/>
-</geometry>
-<material name="grey">
-<color rgba="0.5 0.5 0.5 1.0"/>
-</material>
-</visual>
-<collision>
-<geometry>
-<box size="0.09 0.07 0.535"/>
-</geometry>
-</collision>
-</link>
-<joint name="left_arm_joint" type="fixed">
-<parent link="seat" />
-<child link="left_arm" />
-<origin xyz="0 0.245 0.30" rpy="0 1.0 0"/>
-</joint>
-<link name="right_arm">
-<visual>
-<geometry>
-<box size="0.09 0.07 0.535"/>
-</geometry>
-<material name="grey">
-<color rgba="0.5 0.5 0.5 1.0"/>
-</material>
-</visual>
-<collision>
-<geometry>
-<box size="0.09 0.07 0.535"/>
-</geometry>
-</collision>
-</link>
-<joint name="right_arm_joint" type="fixed">
-<parent link="seat" />
-<child link="right_arm" />
-<origin xyz="0 -0.245 0.30" rpy="0 1.0 0"/>
-</joint>
-<!-- Note: do NOT include lidar here. lidar will be included by robot_top. -->
+<!-- whill_model_cr2: body-only definition (macroized).
+     Place at: <your_package>/urdf/whill_model_cr2.urdf.xacro -->
+<xacro:macro name="whill_body_v0" params="robot_name='whill_model_cr2' gazebo='classic' use_ros2_control='false'" xmlns:xacro="http://ros.org/wiki/xacro">
+  <xacro:arg name="robot_name" default="${robot_name}"/>
+  <xacro:arg name="gazebo" default="${gazebo}"/>
+  <xacro:arg name="use_ros2_control" default="${use_ros2_control}"/>
+  <!-- Base link -->
+  <link name="base_link">
+    <visual>
+      <geometry>
+        <cylinder length="0.2" radius="0.01"/>
+      </geometry>
+      <material name="blue">
+        <color rgba="0.0 0.0 1.0 1.0"/>
+      </material>
+    </visual>
+  </link>
+  <!-- Base floor -->
+  <link name="base_floor">
+    <visual>
+      <geometry>
+        <box size="0.985 0.37 0.03"/>
+      </geometry>
+      <material name="grey">
+        <color rgba="0.5 0.5 0.5 1.0"/>
+      </material>
+    </visual>
+    <collision>
+      <geometry>
+        <box size="0.985 0.37 0.03"/>
+      </geometry>
+    </collision>
+    <inertial>
+      <origin xyz="0 0 0" rpy="0 0 0" />
+      <mass value="30" />
+      <inertia ixx="1.0" ixy="0.0" ixz="0.0"
+               iyy="1.0" iyz="0.0"
+               izz="1.0" />
+    </inertial>
+  </link>
+  <joint name="base_floor_joint" type="fixed">
+    <parent link="base_link" />
+    <child link="base_floor" />
+    <origin xyz="0.3 0 0" rpy="0 0 0"/>
+  </joint>
+  <!-- Left wheel -->
+  <link name="left_wheel">
+    <visual>
+      <geometry>
+        <cylinder length="0.05" radius="0.1325"/>
+      </geometry>
+      <origin xyz="0 0 0" rpy="0 0 0" />
+      <material name="black">
+        <color rgba="0 0 0 1"/>
+      </material>
+    </visual>
+    <collision>
+      <geometry>
+        <cylinder length="0.05" radius="0.1325"/>
+      </geometry>
+      <origin xyz="0 0 0" rpy="0 0 0" />
+    </collision>
+    <inertial>
+      <origin xyz="0 0 0" rpy="0 0 0" />
+      <mass value="1.0" />
+      <inertia ixx="0.01" ixy="0.0" ixz="0.0"
+               iyy="0.01" iyz="0.0"
+               izz="0.01" />
+    </inertial>
+  </link>
+  <!-- Seat -->
+  <link name="seat">
+    <visual>
+      <geometry>
+        <box size="0.30 0.40 0.05"/>
+      </geometry>
+      <material name="grey">
+        <color rgba="0.5 0.5 0.5 1.0"/>
+      </material>
+    </visual>
+    <collision>
+      <geometry>
+        <box size="0.30 0.40 0.05"/>
+      </geometry>
+    </collision>
+    <inertial>
+      <origin xyz="0 0 0" rpy="0 0 0" />
+      <mass value="5.0" />
+      <inertia ixx="0.5" ixy="0.0" ixz="0.0"
+               iyy="0.5" iyz="0.0"
+               izz="0.5" />
+    </inertial>
+  </link>
+  <joint name="seat_joint" type="fixed">
+    <parent link="base_floor" />
+    <child link="seat" />
+    <origin xyz="-0.10 0 0.215" rpy="0 0 0"/>
+  </joint>
+  <!-- Left sensor arm -->
+  <link name="left_sensor_arm">
+    <visual>
+      <geometry>
+        <cylinder length="0.11" radius="0.013"/>
+      </geometry>
+      <material name="grey">
+        <color rgba="0.5 0.5 0.5 1.0"/>
+      </material>
+    </visual>
+    <collision>
+      <geometry>
+        <cylinder length="0.11" radius="0.013"/>
+      </geometry>
+    </collision>
+    <inertial>
+      <origin xyz="0 0 0" rpy="0 0 0" />
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